Commit message: M5-e/Phase C-1 + C-2 + C-3: NEO-M8P bring-up + /fix quality + URDF gnss_link
Brings the u-blox NEO-M8P online on /dev/ttyACM0 and ties it into the
chair's URDF as gnss_link. Receiver is producing 3D-fix /fix at 1 Hz
with 2.17 m observed horizontal scatter (1σ) — already better than
FAST-LIO outdoor drift, which is the prerequisite for Phase C-4
EKF fusion.

Phase C-1: receiver bring-up
  - whill_localization/config/ublox_m8p_rover.yaml — derived from the
    upstream c94_m8p_rover template. The receiver ships with a working
    GPS+GLO+BDS+QZSS EEPROM config and ublox_gps_node's CFG-GNSS
    reconfiguration kept NACK'ing even when we tried to match the
    enable bits. Set config_on_startup: false so the driver opens the
    port read-only against whatever the receiver has persisted. The
    trade-off (dynamic_model, nav_rate, dgnss_mode become inert) is
    captured in the yaml comments — re-enable once we own a clean
    receiver baseline via a u-center factory reset.
  - whill_localization/launch/gnss_launch.py — single ublox_gps_node
    with OnProcessExit shutdown handler so a USB unplug brings the
    launch down cleanly instead of leaving a stale topic graph.

Phase C-2: /fix quality static 60 s
  Chair stationary, antenna relocated from under-chair bucket to the
  footrest for sky view. 54 / 54 samples in 3D FIX, observed 1σ
  horizontal scatter r = 2.17 m, vertical 1.83 m. Receiver self-reported
  1σ is ~10× the observed (20→17 m converging) — a u-blox standalone
  trait that just makes navsat_transform_node weight GPS conservatively.

Phase C-3: gnss_link in URDF
  Added base_link → gnss_link with a magenta cylinder visual. Initial
  offset (0.40, 0.00, -0.10) is the footrest-mount stand-in, marked
  TEMPORARY in the file comment — antenna is not mechanically fixed
  yet and will need re-measurement before Phase C-6 long-distance
  drift verification. xacro expansion verified
  (`xyz="0.4 0.0 -0.1"`).

docs/session-2026-05-30.md
  Appended Phase C-1/C-2/C-3 narrative plus a resume point describing
  the exact next steps for navsat_transform_node integration and
  ekf_map gps0 wiring.

Resume point for the next session: Phase C-4. The recommended
navsat_transform_node settings (use_odometry_yaw: true,
broadcast_utm_transform: false, zero_altitude: true, wait_for_datum:
false) and the rationale (PCMK-G3X orientation field is unavailable,
two_d_mode parity, no NTRIP yet) are spelled out in the session log.

File: src/whill_sensors_bringup/urdf/whill_with_sensors.urdf.xacro (robot description, xacro)
@@ -117,4 +117,25 @@
   <xacro:property name="camera_pitch" value="0.0"/>
   <xacro:property name="camera_yaw"   value="0.0"/>
+  <!-- GNSS antenna (u-blox NEO-M8P) pose in base_link.
+       Phase C-3 (2026-05-30): TEMPORARY placement. The user moved the
+       antenna out of the under-chair bucket and onto the rider's
+       footrest to improve sky view (the bucket roof obscured nearly
+       half the hemisphere). The footrest sits in front of base_link
+       and roughly at floor height, so x ≈ +0.40 m forward, y = 0
+       centerline, z ≈ -0.10 m (just above the ground plane at
+       z=-0.1175 m).
+       The antenna is NOT mechanically fixed yet — these values are
+       a stand-in good to about ±0.1 m. Re-measure with a tape before
+       Phase C-6 (long-distance drift verification). Once a permanent
+       mount is decided, narrow these values and remove this comment.
+       robot_localization's navsat_transform_node absorbs antenna
+       offset error into its EKF covariance, so a rough initial value
+       is acceptable for Phase C-4 wiring. -->
+  <xacro:property name="gnss_x"     value="0.40"/>
+  <xacro:property name="gnss_y"     value="0.0"/>
+  <xacro:property name="gnss_z"     value="-0.10"/>
+  <xacro:property name="gnss_roll"  value="0.0"/>
+  <xacro:property name="gnss_pitch" value="0.0"/>
+  <xacro:property name="gnss_yaw"   value="0.0"/>
   <!-- ====================================================================
        Links and joints
@@ -191,3 +212,23 @@
             rpy="${camera_roll} ${camera_pitch} ${camera_yaw}"/>
   </joint>
+  <!-- GNSS antenna. Visual is a small magenta cylinder so it stands
+       out from imu_link (orange) and the other sensors in RViz.
+       Frame name `gnss_link` matches the frame_id ublox_gps_node
+       stamps on /fix (whill_localization/config/ublox_m8p_rover.yaml). -->
+  <link name="gnss_link">
+    <visual>
+      <geometry>
+        <cylinder length="0.025" radius="0.030"/>
+      </geometry>
+      <material name="gnss_magenta">
+        <color rgba="0.9 0.2 0.7 1.0"/>
+      </material>
+    </visual>
+  </link>
+  <joint name="base_link_to_gnss" type="fixed">
+    <parent link="base_link"/>
+    <child  link="gnss_link"/>
+    <origin xyz="${gnss_x} ${gnss_y} ${gnss_z}"
+            rpy="${gnss_roll} ${gnss_pitch} ${gnss_yaw}"/>
+  </joint>
 </robot>
